File: circuit/receiver/receiver.kicad_pcb (KiCad board)
At the start: 2 copper layers, 56 x 47 mm, 21 parts, among them J1 Conn_01x03_Pin, J2 Conn_01x04_Pin, J3 Conn_02x06_Top_Bottom, U1 74HC4051, U2 74HC4051, U4 ESP32-C3_SUPERMINI_TH

Commit message: refactor: add labels to circuits
Parts:
- removed H1, H2: MountingHole_2.2mm_M2, MountingHole:MountingHole_2.2mm_M2
- added 680 R1: 680, Resistor_THT:R_Axial_DIN0207_L6.3mm_D2.5mm_P10.16mm_Horizontal, B.Cu at (164.8, 50.0)
- added 680 R2: 680, Resistor_THT:R_Axial_DIN0207_L6.3mm_D2.5mm_P10.16mm_Horizontal, B.Cu at (165.0, 52.9)
- added photoMOS 1: AQY212EH, Package_DIP:DIP-4_W7.62mm, B.Cu at (182.0, 69.0)
- added photoMOS 2: AQY212EH, Package_DIP:DIP-4_W7.62mm, B.Cu at (172.9, 76.0)
- 100: renamed from R1; value 1k -> 100
- 104 C1: renamed from C2
- 104 C2: renamed from C1
- 1k: renamed from R8; value 510 -> 1k
- 220: renamed from R2; value 2k -> 220
- 2k: renamed from R5; value 6.8k -> 2k
- 3.3k: renamed from R9; value 330 -> 3.3k
- 330: renamed from R3; value 3.3k -> 330
- 470: renamed from R4; value 4.7k -> 470
- 6.8k: renamed from R6; value 10k -> 6.8k
- J1: footprint Connector_PinHeader_2.54mm:PinHeader_1x03_P2.54mm_Vertical -> Connector_JST:JST_XH_B3B-XH-A_1x03_P2.50mm_Vertical
- J2: footprint Connector_PinHeader_2.54mm:PinHeader_1x04_P2.54mm_Vertical -> Connector_JST:JST_XH_B4B-XH-A_1x04_P2.50mm_Vertical
- MUX 1: renamed from U2
- MUX 2: renamed from U1
- moved J2 3.48 mm to (175.5, 82.2), turned to -90 degrees
- moved J3 1.88 mm to (173.5, 66.6)
- moved J1 1.58 mm to (181.5, 56.5), turned to 90 degrees
- renumbered R11 to 10K, R10 to 10k, R7 to 680
Connections:
- MUX 1 pad 3: Net-(J1-Pin_1) -> Net-(U2-A)
- MUX 2 pad 3: Net-(J1-Pin_2) -> Net-(U1-A)
- U4 pad 8: Net-(J2-Pin_3) -> Net-(J2-Pin_4)
- U4 pad 9: Net-(J2-Pin_4) -> Net-(J2-Pin_3)
Routing:
- net Net-(U1-A): track 0.00 -> 41.3 mm
- net Net-(U2-A): track 0.00 -> 37.9 mm
- net Net-(J1-Pin_2): track 50.8 -> 21.7 mm, vias 1 -> 0
- net Net-(J1-Pin_1): track 32.9 -> 5.71 mm
- net Net-(R13-Pad2): track 0.00 -> 26.9 mm
- net Net-(R12-Pad2): track 0.00 -> 19.5 mm
- net Net-(J3-Pin_1): track 31.5 -> 46.9 mm, vias 1 -> 0
- net Net-(U1-S1): track 71.7 -> 84.7 mm
- net Net-(U1-S0): track 62.1 -> 74.1 mm
- net Net-(U1-S2): track 80.9 -> 69.7 mm
- net Net-(U1-VCC): track 106.9 -> 114.9 mm
- net Net-(U2-~{E}): track 49.9 -> 52.6 mm, vias 0 -> 1
- net Net-(J2-Pin_3): track 8.93 -> 11.4 mm
- net Net-(J2-Pin_4): track 8.93 -> 11.4 mm
- net Net-(U1-A0): track 11.0 -> 12.7 mm
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Other:
- board text added: "1"
- board text added: "2"
- board text added: "A"
- board text added: "B"
- board text added: "Copyright (c) Abhijith Vijayan"
- board text added: "GND"
- board text added: "PUSH"
- board text added: "SWC Receiver v1.1 (rev 1)"
- board text removed: "SWC v1.0 (rev 1)"
